Commit message: Update prm.xacro

File: prm_ws/src/prm_description/urdf/prm.xacro (robot description, xacro)
@@ -1,4 +1,5 @@
 <?xml version="1.0" ?>
 <robot name="prm" xmlns:xacro="http://www.ros.org/wiki/xacro">
+  <!--Raccourcis - similaires a des variabls auxquelles on assigne des valeurs par defaut-->
   <xacro:property name="cameraSize" value="0.05"/>
   <xacro:property name="cameraMass" value="0.00109"/>
@@ -6,8 +7,9 @@
   <xacro:include filename="$(find prm_description)/urdf/materials.xacro" />
   <xacro:include filename="$(find prm_description)/urdf/macros.xacro" />
+<!--Description des objets-->
 <!--Chassis-->
 <link name="base_link">
       <pose>0 0 0.1 0 0 0</pose>
-<inertial>
+  <inertial>
     <origin rpy="0 0 0" xyz="-0.083972 0.064624 0.0325"/>
     <mass value="8"/>
@@ -27,4 +29,5 @@
   </collision>
 </link>
+<!--Entretoises (les 4 sont representees en un fichier .stl pour plus de simplicite de manipulation)-->
 <link name="Lien_PlaqueSup">
   <inertial>
@@ -51,4 +54,5 @@
   <child link="Lien_PlaqueSup"/>
 </joint>
+<!--Plaque superieure-->
 <link name="Plaque_sup">
   <inertial>
@@ -75,5 +79,5 @@
   <child link="Plaque_sup"/>
 </joint>
-<!--Sensors-->
+<!--Capteurs-->
 <!--RPLidar-->
 <link name="laser">

Commit message: Ajout des controlleurs pan et tilt pour la tourelle camera

File: prm_ws/src/prm_description/urdf/prm.xacro (robot description, xacro)
@@ -156,6 +156,16 @@
   <axis xyz="9e-06 -0.0 -0.01"/>
   <limit effort='10000' lower="-1.570796" upper="1.570796" velocity="10000"/>
-    <dynamics damping="100.0" friction="200.0"/>
-</joint>
+    <dynamics damping="0.1" friction="0.2"/> <!--100.0 et 200.0-->
+</joint>
+<transmission name="$pan_trans">
+      <type>transmission_interface/SimpleTransmission</type>
+      <joint name="Pan_joint">
+        <hardwareInterface>EffortJointInterface</hardwareInterface>
+      </joint>
+      <actuator name="$panMotor">
+        <hardwareInterface>EffortJointInterface</hardwareInterface>
+        <mechanicalReduction>1</mechanicalReduction>
+      </actuator>
+</transmission>
 <!--Tourelle Camera - Rotation x-->
 <link name="Tilt">
@@ -184,6 +194,16 @@
   <axis xyz="-0.01 -5.3e-05 -9e-06"/>
   <limit effort='1000' lower="-1.434661" upper="1.434661" velocity="100"/>
-    <dynamics damping="100.0" friction="200.0"/>
-</joint>
+    <dynamics damping="0.1" friction="0.2"/> <!--100.0 et 200.0-->
+</joint>
+<transmission name="$tilt_trans">
+      <type>transmission_interface/SimpleTransmission</type>
+      <joint name="Tilt_joint">
+        <hardwareInterface>EffortJointInterface</hardwareInterface>
+      </joint>
+      <actuator name="$tiltMotor">
+        <hardwareInterface>EffortJointInterface</hardwareInterface>
+        <mechanicalReduction>1</mechanicalReduction>
+      </actuator>
+</transmission>
 <!--Roues-->
 <!--Roue gauche-->

Commit message: Nouveau modele urdf

File: prm_ws/src/prm_description/urdf/prm.xacro (robot description, xacro)
@@ -7,17 +7,17 @@
   <xacro:include filename="$(find prm_description)/urdf/materials.xacro" />
   <xacro:include filename="$(find prm_description)/urdf/macros.xacro" />
-<!--Description des objets-->
+<!--Description des liens-->
 <!--Chassis-->
 <link name="base_link">
-      <pose>0 0 0.1 0 0 0</pose>
-  <inertial>
-    <origin rpy="0 0 0" xyz="-0.083972 0.064624 0.0325"/>
-    <mass value="8"/>
-    <inertia ixx="0.000596" ixy="-0.0" ixz="-0.001035" iyy="0.000385" iyz="0.00104" izz="0.00087"/>
+  <pose>0 0 0.1 0 0 1</pose>
+  <inertial>
+    <origin rpy="0 0 0" xyz="-0.0839777178129331 0.04440645528739363 0.03211202600509656"/>
+    <mass value="0.27584583240478544"/>
+    <inertia ixx="0.001046" ixy="-1e-06" ixz="-0.0" iyy="0.000392" iyz="1.1e-05" izz="0.001324"/>
   </inertial>
   <visual>
     <origin rpy="0 0 0" xyz="0 0 0"/>
     <geometry>
-      <mesh filename="package://prm_description/meshes/base_link_m-binary.stl"/>
+      <mesh filename="package://prm_description/meshes/base_link.stl"/>
     </geometry>
   </visual>
@@ -25,203 +25,73 @@
     <origin rpy="0 0 0" xyz="0 0 0"/>
     <geometry>
-      <mesh filename="package://prm_description/meshes/base_link_m-binary.stl"/>
-    </geometry>
-  </collision>
-</link>
-<!--Entretoises (les 4 sont representees en un fichier .stl pour plus de simplicite de manipulation)-->
-<link name="Lien_PlaqueSup">
-  <inertial>
-    <origin rpy="0 0 0" xyz="-0.04000000000000001 0.060000000000000005 0.029999999999999992"/>
-    <mass value="0.016234"/>
-    <inertia ixx="6.3e-05" ixy="-0.0" ixz="-0.000202" iyy="3.1e-05" iyz="0.000202" izz="8.4e-05"/>
-  </inertial>
-  <visual>
-    <origin rpy="0 0 0" xyz="0.044 -0.008694 -0.051408"/>
-    <geometry>
-      <mesh filename="package://prm_description/meshes/Hexagon_Screw_Nylon_60mm_Through_Hole_1_m-binary.stl"/>
-    </geometry>
-  </visual>
-  <collision>
-    <origin rpy="0 0 0" xyz="0.044 -0.008694 -0.051408"/>
-    <geometry>
-      <mesh filename="package://prm_description/meshes/Hexagon_Screw_Nylon_60mm_Through_Hole_1_m-binary.stl"/>
-    </geometry>
-  </collision>
-</link>
-<joint name="Rigid112" type="fixed">
-  <origin rpy="0 0 0" xyz="-0.044 0.008694 0.051408"/>
-  <parent link="base_link"/>
-  <child link="Lien_PlaqueSup"/>
-</joint>
-<!--Plaque superieure-->
-<link name="Plaque_sup">
-  <inertial>
-    <origin rpy="0 0 0" xyz="-0.04000000000000001 0.060807999999999994 0.0007500000000000007"/>
-    <mass value="0.099139"/>
-    <inertia ixx="0.000271" ixy="0.0" ixz="-0.001707" iyy="0.000189" iyz="0.001707" izz="0.00046"/>
-  </inertial>
-  <visual>
-    <origin rpy="0 0 0" xyz="0.044 -0.008694 -0.111408"/>
-    <geometry>
-      <mesh filename="package://prm_description/meshes/Plaque_sup_1_m-binary.stl"/>
-    </geometry>
-  </visual>
-  <collision>
-    <origin rpy="0 0 0" xyz="0.044 -0.008694 -0.111408"/>
-    <geometry>
-      <mesh filename="package://prm_description/meshes/Plaque_sup_1_m-binary.stl"/>
-    </geometry>
-  </collision>
-</link>
-<joint name="Rigid116" type="fixed">
-  <origin rpy="0 0 0" xyz="0.0 0.0 0.06"/>
-  <parent link="Lien_PlaqueSup"/>
-  <child link="Plaque_sup"/>
-</joint>
-<!--Capteurs-->
-<!--RPLidar-->
-<link name="laser">
-  <inertial>
-    <origin rpy="0 0 0" xyz="0.02745700000000001 -0.040062 0.024728000000000014"/>
-    <mass value="0.073056"/>
-    <inertia ixx="6.2e-05" ixy="1e-06" ixz="-0.001763" iyy="3.2e-05" iyz="0.001757" izz="7.2e-05"/>
-  </inertial>
-  <visual>
-    <origin rpy="0 0 0" xyz="0.112 -0.130239 -0.112908"/>
-    <geometry>
-      <mesh filename="package://prm_description/meshes/RP-lidar-A1_v1_v1_1_m-binary.stl"/>
-    </geometry>
-  </visual>
-  <collision>
-    <origin rpy="0 0 0" xyz="0.112 -0.130239 -0.112908"/>
-    <geometry>
-      <mesh filename="package://prm_description/meshes/RP-lidar-A1_v1_v1_1_m-binary.stl"/>
-    </geometry>
-  </collision>
-</link>
- <joint name="rplidar_joint" type="fixed">
-  <origin rpy="0 0 0" xyz="-0.068 0.121545 0.0015"/>
-  <parent link="Plaque_sup"/>
-  <child link="laser"/>
-</joint>
-<!--CameraRpi-->
-<link name="camera">
-  <inertial>
-    <origin rpy="0 0 0" xyz="-0.0027800000000000047 -0.0006060000000000093 3.899999999999737e-05"/>
-    <mass value="0.00109"/>
-    <inertia ixx="0.0" ixy="0.0" ixz="0.0" iyy="0.0" iyz="-0.0" izz="0.0"/>
-  </inertial>
-  <visual>
-    <origin rpy="0 0 0" xyz="0.081607 0.087487 -0.094501"/>
-    <geometry>
-      <mesh filename="package://prm_description/meshes/RspCameraMia_v1_1_m-binary.stl"/>
-    </geometry>
-  </visual>
-  <collision>
-    <origin rpy="0 0 0" xyz="0.081607 0.087487 -0.094501"/>
-    <geometry>
-      <mesh filename="package://prm_description/meshes/RspCameraMia_v1_1_m-binary.stl"/>
-    </geometry>
-  </collision>
-</link>
-<joint name="Rigid134" type="fixed">
-  <origin rpy="0 0 0" xyz="0.011996 -0.02123 0.012078"/>
-  <parent link="Tilt"/>
-  <child link="camera"/>
-</joint>
-<!--Tourelle Camera - Rotation z-->
-<link name="Pan">
-  <inertial>
-    <origin rpy="0 0 0" xyz="-0.00019700000000000273 -0.006970999999999998 0.013874999999999998"/>
-    <mass value="0.102211"/>
-    <inertia ixx="1.7e-05" ixy="-0.0" ixz="-0.000253" iyy="1.4e-05" iyz="0.000256" izz="1.9e-05"/>
-  </inertial>
-  <visual>
-    <origin rpy="0 0 0" xyz="0.084018 0.039106 -0.051732"/>
-    <geometry>
-      <mesh filename="package://prm_description/meshes/Component32_1_m-binary.stl"/>
-    </geometry>
-  </visual>
-  <collision>
-    <origin rpy="0 0 0" xyz="0.084018 0.039106 -0.051732"/>
-    <geometry>
-      <mesh filename="package://prm_description/meshes/Component32_1_m-binary.stl"/>
-    </geometry>
-  </collision>
-</link>
-<joint name="Pan_joint" type="revolute">
-  <origin rpy="0 0 0" xyz="-0.084018 -0.039106 0.051732"/>
-  <parent link="base_link"/>
-  <child link="Pan"/>
-  <axis xyz="9e-06 -0.0 -0.01"/>
-  <limit effort='10000' lower="-1.570796" upper="1.570796" velocity="10000"/>
-    <dynamics damping="0.1" friction="0.2"/> <!--100.0 et 200.0-->
-</joint>
-<transmission name="$pan_trans">
-      <type>transmission_interface/SimpleTransmission</type>
-      <joint name="Pan_joint">
-        <hardwareInterface>EffortJointInterface</hardwareInterface>
-      </joint>
-      <actuator name="$panMotor">
-        <hardwareInterface>EffortJointInterface</hardwareInterface>
-        <mechanicalReduction>1</mechanicalReduction>
-      </actuator>
-</transmission>
-<!--Tourelle Camera - Rotation x-->
-<link name="Tilt">
-  <inertial>
-    <origin rpy="0 0 0" xyz="0.01253 -0.003738000000000005 0.008108000000000004"/>
-    <mass value="0.083771"/>
-    <inertia ixx="9e-06" ixy="-0.0" ixz="-8.3e-05" iyy="1.2e-05" iyz="8.4e-05" izz="9e-06"/>
-  </inertial>
-  <visual>
-    <origin rpy="0 0 0" xyz="0.093603 0.066257 -0.082423"/>
-    <geometry>
-      <mesh filename="package://prm_description/meshes/Component31_1_m-binary.stl"/>
-    </geometry>
-  </visual>
-  <collision>
-    <origin rpy="0 0 0" xyz="0.093603 0.066257 -0.082423"/>
-    <geometry>
-      <mesh filename="package://prm_description/meshes/Component31_1_m-binary.stl"/>
-    </geometry>
-  </collision>
-</link>
-<joint name="Tilt_joint" type="revolute">
-  <origin rpy="0 0 0" xyz="-0.009585 -0.027151 0.030691"/>
-  <parent link="Pan"/>
-  <child link="Tilt"/>
-  <axis xyz="-0.01 -5.3e-05 -9e-06"/>
-  <limit effort='1000' lower="-1.434661" upper="1.434661" velocity="100"/>
-    <dynamics damping="0.1" friction="0.2"/> <!--100.0 et 200.0-->
-</joint>
-<transmission name="$tilt_trans">
-      <type>transmission_interface/SimpleTransmission</type>
-      <joint name="Tilt_joint">
-        <hardwareInterface>EffortJointInterface</hardwareInterface>
-      </joint>
-      <actuator name="$tiltMotor">
-        <hardwareInterface>EffortJointInterface</hardwareInterface>
-        <mechanicalReduction>1</mechanicalReduction>
-      </actuator>
-</transmission>
-<!--Roues-->
+      <mesh filename="package://prm_description/meshes/base_link.stl"/>
+    </geometry>
+  </collision>
+</link>
+<!--Roue Folle-->
+<!--Roue Folle - Rotation z-->
+<link name='stem'>
+  <inertial>
+    <mass value="0.008"/>
+    <inertia ixx="0.0" ixy="0.0" ixz="-1e-05" iyy="0.0" iyz="1e-05" izz="0.0"/>
+  </inertial>
+  <collision>
+    <geometry>
+      <cylinder radius='0.010319' length='0.003408'/>
+    </geometry>
+  </collision>
+  <visual>
+    <geometry>
+      <cylinder radius='0.010319' length='0.003408'/>
+    </geometry>
+  </visual>
+</link>
+<joint name="stem_joint" type="fixed">
+  <origin rpy="0 0 0" xyz="-0.084 0.13815 0.011704"/>
+  <parent link="base_link"/>
+  <child link="stem"/>
+   <axis xyz="0 0 1"/>
+  <limit effort="100000000" velocity="100000000"/>
+</joint>
+<!--Roue Folle - Rotation x-->
+<link name='caster'>
+  <inertial>
+    <mass value="0.008419"/>
+    <inertia ixx="0.000135796" ixy="0.0" ixz="0.0" iyy="0.000135796" iyz="0.0" izz="0.000135796"/>
+  </inertial>
+  <collision>
+    <geometry>
+      <sphere radius='0.005852'/>
+    </geometry>
+  </collision>
+  <visual>
+    <geometry>
+      <sphere radius='0.005852'/>
+    </geometry>
+  </visual>
+</link>
+<joint name="caster_joint" type="fixed">
+  <origin rpy="0 0 0" xyz="0 0 -0.007"/>
+  <parent link="stem"/>
+  <child link="caster"/>
+   <limit effort="100000000" velocity="100000000"/>
+</joint>
 <!--Roue gauche-->
-<link name="Left_Wheel_1">
-  <inertial>
-    <origin rpy="0 0 0" xyz="0.016849000000000003 4.999999999999796e-06 7.000000000000062e-06"/>
-    <mass value="0.1"/>
-    <inertia ixx="3e-05" ixy="-0.0" ixz="-2.6e-05" iyy="1.9e-05" iyz="2.6e-05" izz="1.9e-05"/>
-  </inertial>
-  <visual>
-    <origin rpy="0 0 0" xyz="0.029 -0.002194 -0.0325"/>
-    <geometry>
-      <mesh filename="package://prm_description/meshes/Left_Wheel_1_m-binary.stl"/>
-    </geometry>
-  </visual>
-  <collision>
-    <origin rpy="1.5707 1.5707 1.5707" xyz="0.016 0 0"/>
-    <geometry>
-      <cylinder radius="0.0325" length='0.026'/>
+<link name="left_wheel_1">
+  <inertial>
+    <origin rpy="0 0 0" xyz="0.016848728056798892 5.266257451158347e-06 7.513062202278709e-06"/>
+    <mass value="0.05572555972770472"/>
+    <inertia ixx="3e-05" ixy="-0.0" ixz="-0.0" iyy="1.9e-05" iyz="-0.0" izz="1.9e-05"/>
+  </inertial>
+  <visual>
+    <origin rpy="0 0 0" xyz="0.029 -0.002194 -0.032408"/>
+    <geometry>
+      <mesh filename="package://prm_description/meshes/left_wheel_1.stl"/>
+    </geometry>
+  </visual>
+  <collision>
+    <origin rpy="0 0 0" xyz="0.029 -0.002194 -0.032408"/>
+    <geometry>
+      <mesh filename="package://prm_description/meshes/left_wheel_1.stl"/>
     </geometry>
       <surface>
@@ -235,39 +105,21 @@
   </collision>
 </link>
-<joint name="Rev121" type="continuous">
-  <origin rpy="0 0 0" xyz="-0.029 0.002194 0.0325"/>
-  <parent link="base_link"/>
-  <child link="Left_Wheel_1"/>
-   <axis xyz="1 0 0"/>
-    <limit effort="100" velocity="100"/>
-    <joint_properties damping="0" friction="0"/>
-</joint>
-<transmission name="lw_trans">
-      <type>transmission_interface/SimpleTransmission</type>
-      <joint name="Rev121">
-        <hardwareInterface>EffortJointInterface</hardwareInterface>
-      </joint>
-      <actuator name="$lwMotor">
-        <hardwareInterface>EffortJointInterface</hardwareInterface>
-        <mechanicalReduction>10</mechanicalReduction>
-      </actuator>
-</transmission>
 <!--Roue droite-->
-<link name="Right_Wheel_3">
-  <inertial>
-    <origin rpy="0 0 0" xyz="-0.016839999999999994 -7.000000000000062e-06 4.9999999999980616e-06"/>
-    <mass value="0.1"/>
-    <inertia ixx="3e-05" ixy="0.0" ixz="-0.000285" iyy="1.9e-05" iyz="0.000285" izz="1.9e-05"/>
+<link name="right_wheel_3">
+  <inertial>
+    <origin rpy="0 0 0" xyz="-0.01683997258297837 -7.067395580239062e-06 5.538351484139781e-06"/>
+    <mass value="0.055725588971055603"/>
+    <inertia ixx="3e-05" ixy="0.0" ixz="-0.0" iyy="1.9e-05" iyz="0.0" izz="1.9e-05"/>
   </inertial>
   <visual>
     <origin rpy="0 0 0" xyz="0.139 -0.002194 -0.032408"/>
     <geometry>
-      <mesh filename="package://prm_description/meshes/Right_Wheel_3_m-binary.stl"/>
-    </geometry>
-  </visual>
-  <collision>
-    <origin rpy="1.5707 1.5707 1.5707" xyz="-0.016 0 0"/>
-    <geometry>
-      <cylinder radius="0.0325" length='0.026'/>
+      <mesh filename="package://prm_description/meshes/right_wheel_3.stl"/>
+    </geometry>
+  </visual>
+  <collision>
+    <origin rpy="0 0 0" xyz="0.139 -0.002194 -0.032408"/>
+    <geometry>
+      <mesh filename="package://prm_description/meshes/right_wheel_3.stl"/>
     </geometry>
       <surface>
@@ -281,69 +133,220 @@
   </collision>
 </link>
-<joint name="Rev120" type="continuous">
-  <origin rpy="0 0 0" xyz="-0.139 0.002194 0.0325"/>
-  <parent link="base_link"/>
-  <child link="Right_Wheel_3"/>
-  <axis xyz="1 0 0"/>
-    <limit effort="100" velocity="100"/>
-    <dynamics damping="0.0" friction="0.0"/>
-</joint>
-<transmission name="$rw_trans">
-      <type>transmission_interface/SimpleTransmission</type>
-      <joint name="Rev120">
-        <hardwareInterface>EffortJointInterface</hardwareInterface>
-      </joint>
-      <actuator name="$rwMotor">
-        <hardwareInterface>EffortJointInterface</hardwareInterface>
-        <mechanicalReduction>10</mechanicalReduction>
-      </actuator>
+<!--Entretoises (les 4 sont representees en un fichier .stl pour plus de simplicite de manipulation)-->
+<link name="lien_plaque_sup_1">
+  <inertial>
+    <origin rpy="0 0 0" xyz="-0.039999999999991334 0.06000009548239064 0.03000032830658448"/>
+    <mass value="0.016233798346575297"/>
+    <inertia ixx="6.3e-05" ixy="-0.0" ixz="0.0" iyy="3.1e-05" iyz="-0.0" izz="8.4e-05"/>
+  </inertial>
+  <visual>
+    <origin rpy="0 0 0" xyz="0.044 -0.008694 -0.051408"/>
+    <geometry>
+      <mesh filename="package://prm_description/meshes/lien_plaque_sup_1.stl"/>
+    </geometry>
+  </visual>
+  <collision>
+    <origin rpy="0 0 0" xyz="0.044 -0.008694 -0.051408"/>
+    <geometry>
+      <mesh filename="package://prm_description/meshes/lien_plaque_sup_1.stl"/>
+    </geometry>
+  </collision>
+</link>
+<!--Plaque superieure-->
+<link name="plaque_sup_1">
+  <inertial>
+    <origin rpy="0 0 0" xyz="-0.03999999999999 0.060785568215751755 0.000750328306584766"/>
+    <mass value="0.09905330487184344"/>
+    <inertia ixx="0.000271" ixy="-0.0" ixz="-0.0" iyy="0.000189" iyz="0.0" izz="0.000459"/>
+  </inertial>
+  <visual>
+    <origin rpy="0 0 0" xyz="0.044 -0.008694 -0.111408"/>
+    <geometry>
+      <mesh filename="package://prm_description/meshes/plaque_sup_1.stl"/>
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
Commit message: Correction erreur taille Lidar

File: prm_ws/src/prm_description/urdf/prm.xacro (robot description, xacro)
@@ -183,5 +183,5 @@
     <origin rpy="0 0 0" xyz="0.112 -0.130239 -0.112908"/>
     <geometry>
-      <mesh filename="package://prm_description/meshes/laser_1.stl" scale="0.001 0.001 0.001"/>
+      <mesh filename="package://prm_description/meshes/laser_1.stl"/>
     </geometry>
   </visual>
@@ -189,5 +189,5 @@
     <origin rpy="0 0 0" xyz="0.112 -0.130239 -0.112908"/>
     <geometry>
-      <mesh filename="package://prm_description/meshes/laser_1.stl" scale="0.001 0.001 0.001"/>
+      <mesh filename="package://prm_description/meshes/laser_1.stl"/>
     </geometry>
   </collision>
