Commit message: Changement d'unites en mm

File: prm_ws/src/prm_description/urdf/prm.xacro (robot description, xacro)
@@ -19,5 +19,5 @@
     <origin rpy="0 0 0" xyz="0 0 0"/>
     <geometry>
-      <mesh filename="package://prm_description/meshes/base_link.stl"/>
+      <mesh filename="package://prm_description/meshes/base_link.stl" scale="0.001 0.001 0.001"/>
     </geometry>
   </visual>
@@ -25,5 +25,5 @@
     <origin rpy="0 0 0" xyz="0 0 0"/>
     <geometry>
-      <mesh filename="package://prm_description/meshes/base_link.stl"/>
+      <mesh filename="package://prm_description/meshes/base_link.stl" scale="0.001 0.001 0.001"/>
     </geometry>
   </collision>
@@ -87,5 +87,5 @@
     <origin rpy="0 0 0" xyz="0.029 -0.002194 -0.032408"/>
     <geometry>
-      <mesh filename="package://prm_description/meshes/left_wheel_1.stl"/>
+      <mesh filename="package://prm_description/meshes/left_wheel_1.stl" scale="0.001 0.001 0.001"/>
     </geometry>
   </visual>
@@ -93,5 +93,5 @@
     <origin rpy="0 0 0" xyz="0.029 -0.002194 -0.032408"/>
     <geometry>
-      <mesh filename="package://prm_description/meshes/left_wheel_1.stl"/>
+      <mesh filename="package://prm_description/meshes/left_wheel_1.stl" scale="0.001 0.001 0.001"/>
     </geometry>
       <surface>
@@ -115,5 +115,5 @@
     <origin rpy="0 0 0" xyz="0.139 -0.002194 -0.032408"/>
     <geometry>
-      <mesh filename="package://prm_description/meshes/right_wheel_3.stl"/>
+      <mesh filename="package://prm_description/meshes/right_wheel_3.stl" scale="0.001 0.001 0.001"/>
     </geometry>
   </visual>
@@ -121,5 +121,5 @@
     <origin rpy="0 0 0" xyz="0.139 -0.002194 -0.032408"/>
     <geometry>
-      <mesh filename="package://prm_description/meshes/right_wheel_3.stl"/>
+      <mesh filename="package://prm_description/meshes/right_wheel_3.stl" scale="0.001 0.001 0.001"/>
     </geometry>
       <surface>
@@ -143,5 +143,5 @@
     <origin rpy="0 0 0" xyz="0.044 -0.008694 -0.051408"/>
     <geometry>
-      <mesh filename="package://prm_description/meshes/lien_plaque_sup_1.stl"/>
+      <mesh filename="package://prm_description/meshes/lien_plaque_sup_1.stl" scale="0.001 0.001 0.001"/>
     </geometry>
   </visual>
@@ -149,5 +149,5 @@
     <origin rpy="0 0 0" xyz="0.044 -0.008694 -0.051408"/>
     <geometry>
-      <mesh filename="package://prm_description/meshes/lien_plaque_sup_1.stl"/>
+      <mesh filename="package://prm_description/meshes/lien_plaque_sup_1.stl" scale="0.001 0.001 0.001"/>
     </geometry>
   </collision>
@@ -163,5 +163,5 @@
     <origin rpy="0 0 0" xyz="0.044 -0.008694 -0.111408"/>
     <geometry>
-      <mesh filename="package://prm_description/meshes/plaque_sup_1.stl"/>
+      <mesh filename="package://prm_description/meshes/plaque_sup_1.stl" scale="0.001 0.001 0.001"/>
     </geometry>
   </visual>
@@ -169,5 +169,5 @@
     <origin rpy="0 0 0" xyz="0.044 -0.008694 -0.111408"/>
     <geometry>
-      <mesh filename="package://prm_description/meshes/plaque_sup_1.stl"/>
+      <mesh filename="package://prm_description/meshes/plaque_sup_1.stl" scale="0.001 0.001 0.001"/>
     </geometry>
   </collision>
@@ -183,5 +183,5 @@
     <origin rpy="0 0 0" xyz="0.112 -0.130239 -0.112908"/>
     <geometry>
-      <mesh filename="package://prm_description/meshes/laser_1.stl"/>
+      <mesh filename="package://prm_description/meshes/laser_1.stl" scale="0.001 0.001 0.001"/>
     </geometry>
   </visual>
@@ -189,5 +189,5 @@
     <origin rpy="0 0 0" xyz="0.112 -0.130239 -0.112908"/>
     <geometry>
-      <mesh filename="package://prm_description/meshes/laser_1.stl"/>
+      <mesh filename="package://prm_description/meshes/laser_1.stl" scale="0.001 0.001 0.001"/>
     </geometry>
   </collision>
@@ -203,5 +203,5 @@
     <origin rpy="0 0 0" xyz="0.093603 0.066257 -0.082423"/>
     <geometry>
-      <mesh filename="package://prm_description/meshes/tilt_1.stl"/>
+      <mesh filename="package://prm_description/meshes/tilt_1.stl" scale="0.001 0.001 0.001"/>
     </geometry>
   </visual>
@@ -209,5 +209,5 @@
     <origin rpy="0 0 0" xyz="0.093603 0.066257 -0.082423"/>
     <geometry>
-      <mesh filename="package://prm_description/meshes/tilt_1.stl"/>
+      <mesh filename="package://prm_description/meshes/tilt_1.stl" scale="0.001 0.001 0.001"/>
     </geometry>
   </collision>
@@ -223,5 +223,5 @@
     <origin rpy="0 0 0" xyz="0.081607 0.087487 -0.094501"/>
     <geometry>
-      <mesh filename="package://prm_description/meshes/camera_1.stl"/>
+      <mesh filename="package://prm_description/meshes/camera_1.stl" scale="0.001 0.001 0.001"/>
     </geometry>
   </visual>
@@ -229,5 +229,5 @@
     <origin rpy="0 0 0" xyz="0.081607 0.087487 -0.094501"/>
     <geometry>
-      <mesh filename="package://prm_description/meshes/camera_1.stl"/>
+      <mesh filename="package://prm_description/meshes/camera_1.stl" scale="0.001 0.001 0.001"/>
     </geometry>
   </collision>
@@ -243,5 +243,5 @@
     <origin rpy="0 0 0" xyz="0.084018 0.039106 -0.051732"/>
     <geometry>
-      <mesh filename="package://prm_description/meshes/pan_1.stl"/>
+      <mesh filename="package://prm_description/meshes/pan_1.stl" scale="0.001 0.001 0.001"/>
     </geometry>
   </visual>
@@ -249,5 +249,5 @@
     <origin rpy="0 0 0" xyz="0.084018 0.039106 -0.051732"/>
     <geometry>
-      <mesh filename="package://prm_description/meshes/pan_1.stl"/>
+      <mesh filename="package://prm_description/meshes/pan_1.stl" scale="0.001 0.001 0.001"/>
     </geometry>
   </collision>

Commit message: Ajout de README et orientation de la camera

File: prm_ws/src/prm_description/urdf/prm.xacro (robot description, xacro)
@@ -327,5 +327,5 @@
 <!--Joint Camera-->
 <joint name="rigid_camera" type="fixed">
-  <origin rpy="0 0 0" xyz="0.011996 -0.02123 0.012078"/>
+  <origin rpy="0 0 -1.57" xyz="0.011996 -0.02123 0.012078"/> <!--rpy="0 0 -1.57" ajuste l'orientation de la camera-->
   <parent link="tilt_1"/>
   <child link="camera_1"/>
